File: CapSorting/SolenoidProtectionCircuit.sch (KiCad schematic (older format))
At the start: 15 parts, among them CN12 S6B-XH-A, Q1 2SA1015, Q12 2SA1015, Q13 IRLB8721PBF, Q2 IRLB8721PBF

Commit message: 引き直し
Parts:
- removed CN12: S6B-XH-A, JST:S6B-XH-A, symbol SolenoidProtectionCircuit:S6B-XH-A
- added J11: Conn_01x06, Connector_JST:JST_XH_S6B-XH-A_1x06_P2.50mm_Horizontal, symbol Connector_Generic:Conn_01x06
- Q13, Q2: footprint Package_TO_SOT_THT:TO-220-3_Vertical -> CapSorting:IRLB8721PBF-2
Changed lines of the file:
@@
 F 0 "Q13" H 5850 2950 50  0000 L CNN
 F 1 "IRLB8721PBF" H 5850 2850 50  0000 L CNN
-F 2 "Package_TO_SOT_THT:TO-220-3_Vertical" H 5900 2625 50  0001 L CIN
+F 2 "CapSorting:IRLB8721PBF-2" H 5900 2625 50  0001 L CIN
 F 3 "http://www.infineon.com/dgdl/irlb8721pbf.pdf?fileId=5546d462533600a40153566056732591" H 5650 2700 50  0001 L CNN
 	1    5650 2700
@@
 F 0 "Q2" H 5800 5850 50  0000 L CNN
 F 1 "IRLB8721PBF" H 5800 5750 50  0000 L CNN
-F 2 "Package_TO_SOT_THT:TO-220-3_Vertical" H 5850 5525 50  0001 L CIN
+F 2 "CapSorting:IRLB8721PBF-2" H 5850 5525 50  0001 L CIN
 F 3 "http://www.infineon.com/dgdl/irlb8721pbf.pdf?fileId=5546d462533600a40153566056732591" H 5600 5600 50  0001 L CNN
 	1    5600 5600
@@
 Wire Wire Line
 	5700 5800 5700 6100
-$Comp
-L SolenoidProtectionCircuit:S6B-XH-A CN12
-U 1 1 5FE4D0C3
-P 1650 1800
-F 0 "CN12" H 1362 2375 50  0000 C CNN
-F 1 "S6B-XH-A" H 1362 2284 50  0000 C CNN
-F 2 "JST:S6B-XH-A" H 1150 1450 50  0001 C CNN
-F 3 "" H 1150 1450 50  0001 C CNN
-	1    1650 1800
-	1    0    0    -1
-$EndComp
 $Comp
 L power:+24V #PWR0104
@@
 Wire Wire Line
 	1750 1450 1750 2150
+$Comp
+L Connector_Generic:Conn_01x06 J11
+U 1 1 5FE4D6A7
+P 1450 1650
+F 0 "J11" H 1368 2067 50  0000 C CNN
+F 1 "Conn_01x06" H 1368 1976 50  0000 C CNN
+F 2 "Connector_JST:JST_XH_S6B-XH-A_1x06_P2.50mm_Horizontal" H 1450 1650 50  0001 C CNN
+F 3 "~" H 1450 1650 50  0001 C CNN
+	1    1450 1650
+	-1   0    0    -1
+$EndComp
 $EndSCHEMATC
